Commit message: added some urdf stuff to ipynb

File: arm.urdf (robot description, URDF)
Before this commit: robot 5dof_arm_base, 6 links, 5 joints
Joints:
- joint rotating_joint: type continuous -> revolute

Commit message: new urdf

File: arm.urdf (robot description, URDF)
Before this commit: robot 5dof_arm_base, 6 links, 5 joints
Links:
- link elbow_link: geometry collision box size=3 1 7.375; visual box size=3 1 7.375
- link shoulder_link: geometry collision box size=3 1 5.75; visual box size=3 1 5.75
- link wristp_link: geometry collision box size=2 1 2.5; visual box size=2 1 2.5
- link wristr_link: geometry collision box size=1.25 .75 2; visual box size=1.25 .75 2
Joints:
- joint elbow_joint: origin xyz=0 0 6 rpy=0 0 0 -> xyz=0 0 5.75 rpy=0 0 0
- joint wristp_joint: origin xyz=0 0 7.5 rpy=0 0 0 -> xyz=0 0 7.375 rpy=0 0 0

Commit message: works! but not accurate
sdfds

File: arm.urdf (robot description, URDF)
Before this commit: robot 5dof_arm_base, 6 links, 5 joints
Joints:
- joint wristp_joint: limit lower=-1.57 upper=1.57 effort=10 velocity=1.57 -> lower=-1.9 upper=1.57 effort=10 velocity=1.57

Commit message: fixed shoulder degree limit

File: arm.urdf (robot description, URDF)
Before this commit: robot 5dof_arm_base, 6 links, 5 joints
Joints:
- joint shoulder_joint: limit lower=-1.57 upper=1.57 effort=10 velocity=1.57 -> lower=-2.00713 upper=1.57 effort=10 velocity=1.57
